File: midiori.sch (KiCad schematic (older format))
At the start: 51 parts, among them J1 x68000_expansion, J2 DIN-5_180degree, J3 DIN-5_180degree, J4 DIN-5_180degree, J5 AudioJack3, J6 AudioJack3, J7 AudioJack3, U1 74LS245, U10 74LS393, U11 74LS74, U12 74LS30, U13 H11L1, U14 7407, U15 74LS157, U2 74LS27, U3 74LS30, U4 74LS08, U5 74LS38, U6 ym3802-x, U7 74LS32, U8 74LS04, U9 74LS10, X1 16MHz, X2 4.9152MHz

Commit message: PCB layout of fpga version
Parts:
- removed J2, J4: DIN-5_180degree, x68k:sds-50j, symbol Connector:DIN-5_180degree
- removed J5, J6: AudioJack3, Connector_Audio:Jack_3.5mm_CUI_SJ1-3533NG_Horizontal, symbol Connector:AudioJack3
- removed JP1: Jumper_3_Bridged12, Connector_PinHeader_2.54mm:PinHeader_1x03_P2.54mm_Vertical, symbol Jumper:Jumper_3_Bridged12
- removed JP2: Jumper_NO_Small, Connector_PinHeader_2.54mm:PinHeader_1x02_P2.54mm_Vertical, symbol Device:Jumper_NO_Small
- removed R28: 270, Resistor_SMD:R_0805_2012Metric_Pad1.15x1.40mm_HandSolder, symbol Device:R
- removed R29, R7, R8: 220, Resistor_SMD:R_0805_2012Metric_Pad1.15x1.40mm_HandSolder, symbol Device:R
- removed R4, R5: 10K, Resistor_SMD:R_0805_2012Metric_Pad1.15x1.40mm_HandSolder, symbol Device:R
- removed U1: 74LS245, Package_SO:SOIC-20W_7.5x12.8mm_P1.27mm, symbol 74xx:74LS245
- removed U10: 74LS393, Package_SO:SOIC-14_3.9x8.7mm_P1.27mm, symbol 74xx:74LS393
- removed U11: 74LS74, Package_SO:SOIC-14_3.9x8.7mm_P1.27mm, symbol 74xx:74LS74
- removed U12: 74LS30, Package_SO:SOIC-14_3.9x8.7mm_P1.27mm, symbol 74xx:74LS30
- removed U13: H11L1, Package_DIP:DIP-6_W8.89mm_SMDSocket_LongPads, symbol Isolator:H11L1
- removed U14: 7407, Package_SO:SOIC-14_3.9x8.7mm_P1.27mm, symbol 74xx_IEEE:7407
- removed U15: 74LS157, Package_SO:SOIC-16_3.9x9.9mm_P1.27mm, symbol 74xx:74LS157
- removed U2: 74LS27, Package_SO:SOIC-14_3.9x8.7mm_P1.27mm, symbol 74xx:74LS27
- removed U3: 74LS30, symbol 74xx:74LS30
- removed U4: 74LS08, symbol 74xx:74LS08
- removed U5: 74LS38, Package_SO:SOIC-14_3.9x8.7mm_P1.27mm, symbol 74xx:74LS38
- removed U6: ym3802-x, Package_DIP:DIP-40_W15.24mm_Socket, symbol midiori-rescue:ym3802-x-x68k-midiori-rescue
- removed U7: 74LS32, Package_SO:SOIC-14_3.9x8.7mm_P1.27mm, symbol 74xx:74LS32
- removed U8: 74LS04, symbol 74xx:74LS04
- removed U9: 74LS10, Package_SO:SOIC-14_3.9x8.7mm_P1.27mm, symbol 74xx:74LS10
- removed X2: 4.9152MHz, Oscillator:Oscillator_SMD_SeikoEpson_SG8002CA-4Pin_7.0x5.0mm, symbol x68k:SG5032CAN
- added C15, C18, C19, C20, C21, C22, C23: 0.1uF, Capacitor_SMD:C_0805_2012Metric, symbol Device:C
- added C2: 4.7uF, Capacitor_SMD:C_0805_2012Metric, symbol Device:C
- added H1, H2: MountingHole, symbol Mechanical:MountingHole
- added J2: Conn_ARM_JTAG_SWD_10, Connector_PinHeader_1.27mm:PinHeader_2x05_P1.27mm_Vertical_SMD, symbol Connector:Conn_ARM_JTAG_SWD_10
- added R2: 1, Resistor_SMD:R_0805_2012Metric, symbol Device:R
- added U1: 74LCX07, Package_SO:SOIC-14_3.9x8.7mm_P1.27mm, symbol 74xx:74LCX07
- added U10: ICE40HX1K-VQ100, ICE40HX1K-VQ100:QFP50P1600X1600X120-100N, symbol ICE40HX1K-VQ100:ICE40HX1K-VQ100
- added U11: TPS76933, Package_TO_SOT_SMD:SOT-23-5, symbol Regulator_Linear:TPS76933
- added U2: AT25SF081-SSHD-X, Package_SO:SOIC-8_3.9x4.9mm_P1.27mm, symbol Memory_Flash:AT25SF081-SSHD-X
- added U3: TPS76912, Package_TO_SOT_SMD:SOT-23-5, symbol Regulator_Linear:TPS76912
- added U4, U5, U6, U7, U8, U9: SN74LVC8T245DWR, Package_SO:SOIC-24W_7.5x15.4mm_P1.27mm, symbol SN74LVC8T245DWR:SN74LVC8T245DWR
- C1: value u1 -> 4.7uF; footprint Capacitor_SMD:C_0805_2012Metric_Pad1.15x1.40mm_HandSolder -> Capacitor_SMD:C_0805_2012Metric
- C10, C11, C12, C13, C14, C16, C17, C3, C4, C5, C6, C7, C9: value u1 -> 0.1uF; footprint Capacitor_SMD:C_0805_2012Metric_Pad1.15x1.40mm_HandSolder -> Capacitor_SMD:C_0805_2012Metric
- C8: value u1 -> 0.1uF
- J1: symbol midiori-rescue:x68000_expansion-x68k-midiori-rescue -> x68k:x68000_expansion
- R1: value 10K -> 1; footprint Resistor_SMD:R_0805_2012Metric_Pad1.15x1.40mm_HandSolder -> Resistor_SMD:R_0805_2012Metric
- R3: footprint Resistor_SMD:R_0805_2012Metric_Pad1.15x1.40mm_HandSolder -> Resistor_SMD:R_0805_2012Metric
Connections:
- net +5V: now also C15.1, U11.1 (IN), U4.1 (VCCA), U5.1 (VCCA), U6.1 (VCCA), U7.1 (VCCA), U8.1 (VCCA), U9.1 (VCCA); no longer C1.1, C10.1, C12.1, C14.1, C16.1, C17.1, C3.1, C5.1, C7.1, C8.1, R1.1, R3.1, X1.1 (OE), X1.4 (V+)
- net 10MHz: now also U8.3 (A1)
- net A: now also U8.8 (A6)
- net AB1: now also U4.10 (A8)
- net AB10: now also U5.8 (A6)
- net AB11: now also U5.7 (A5)
- net AB12: now also U5.6 (A4)
- net AB13: now also U5.5 (A3)
- net AB14: now also U5.4 (A2)
- net AB15: now also U5.3 (A1)
- net AB16: now also U6.10 (A8)
- net AB17: now also U6.9 (A7)
- net AB18: now also U6.8 (A6)
- net AB19: now also U6.7 (A5)
- net AB2: now also U4.9 (A7)
- net AB20: now also U6.6 (A4)
- net AB21: now also U6.5 (A3)
- net AB22: now also U6.4 (A2)
- net AB23: now also U6.3 (A1)
- net AB3: now also U4.8 (A6)
- net AB4: now also U4.7 (A5)
- net AB5: now also U4.6 (A4)
- net AB6: now also U4.5 (A3)
- net AB7: now also U4.4 (A2)
- net AB8: now also U5.10 (A8)
- net AB9: now also U5.9 (A7)
- net AS: now also U8.7 (A5)
- net B: now also U8.9 (A7)
- net C: now also U8.10 (A8)
- net DB0: now also U7.10 (A8)
- net DB1: now also U7.9 (A7)
- net DB2: now also U7.8 (A6)
- net DB3: now also U7.7 (A5)
- net DB4: now also U7.6 (A4)
- net DB5: now also U7.5 (A3)
- net DB6: now also U7.4 (A2)
- net DB7: now also U7.3 (A1)
- net DTACK: now also U1.6
- net EXRESET: now also U8.4 (A2)
- net GND: now also C12.2, C15.2, C18.2, C19.2, C20.2, C21.2, C22.2, C23.2, J2.3 (GND), J2.5 (GND), J2.9 (GNDDetect), U10.17 (GND), U10.23 (GND), U10.32 (GND), U10.39 (GND), U10.47 (GND), U10.5 (GND), U10.55 (GND), U10.70 (GND), U10.84 (GND), U10.98 (GND), U2.4 (GND), U4.11 (GND), U4.12 (GND), U4.13 (GND), U5.11 (GND), U5.12 (GND), U5.13 (GND), U6.12 (GND), U6.13 (GND), U7.11 (GND), U7.12 (GND), U7.13 (GND), U8.11 (GND), U8.12 (GND), U8.13 (GND), U9.11 (GND), U9.12 (GND), U9.13 (GND); no longer C1.2
- net IACK2: now also U9.3 (A1)
- net IACK4: now also U9.4 (A2)
- net IDDIR: now also U7.2 (DIR), U9.5 (A3)
- net IRQ2: now also U1.2
- net IRQ4: now also U1.4
- net LDS: now also U8.6 (A4)
- net RW: now also U8.5 (A3)
- net at R1.2: now also R2.2, U11.2 (GND), U11.3 (~EN~), U3.2 (GND), U3.3 (~EN~)
- net +3V3: now reaches R3.2
- net +3V3: now also C1.1, C10.1, C12.1, C14.1, C17.1, C3.1, C5.1, C7.1, C8.1, X1.1 (OE), X1.4 (V+), C19.1, C21.1, C23.1, J2.1 (VCC), U10.14 (VCCIO_3), U10.22 (VCCIO_3), U10.31 (VCCIO_2), U10.38 (VCCIO_2), U10.50 (VCC_SPI), U10.58 (VCCIO_1), U10.6 (VCCIO_3), U10.67 (VCCIO_1), U10.75 (VPP_2V5), U10.88 (VCCIO_0), U10.92 (VCCIO_0), U11.5 (OUT), U2.3 (~WP~/IO2), U2.7 (~HOLD~/IO3), U2.8 (VCC), U3.1 (IN), U4.23 (VCCB), U4.24 (VCCB), U5.23 (VCCB), U5.24 (VCCB), U6.23 (VCCB), U6.24 (VCCB), U7.23 (VCCB), U7.24 (VCCB), U8.23 (VCCB), U8.24 (VCCB), U9.23 (VCCB), U9.24 (VCCB)
- net at X1.3 (OUT): now also U10.63 (IOR_61_GBIN2)
- net at R9.2: now also U1.8
- new net: U1.9, U10.66 (IOR_65)
- new net: C1.2, R1.1
- new net: C2.2, R2.1
- new net +1V2: C16.1, C18.1, C2.1, C20.1, C22.1, U10.11 (VCC), U10.35 (VCC), U10.61 (VCC), U10.77 (VCC), U3.5 (OUT)
- new net 10m: U10.97 (IOT_91), U8.21 (B1)
- new net a: U10.3 (IOL_2A), U8.16 (B6)
- new net a1: U10.40 (IOB_41), U4.14 (B8)
- new net a16: U10.71 (IOR_69), U6.14 (B8)
- new net a17: U10.72 (IOR_70), U6.15 (B7)
- new net a18: U10.73 (IOR_71), U6.16 (B6)
- new net a19: U10.74 (IOR_72), U6.17 (B5)
- new net a2: U10.37 (IOB_37), U4.15 (B7)
- new net a20: U10.78 (IOT_73), U6.18 (B4)
- new net a21: U10.79 (IOT_74), U6.19 (B3)
- new net a22: U10.80 (IOT_75), U6.20 (B2)
- new net a23: U10.81 (IOT_77), U6.21 (B1)
- new net a3: U10.34 (IOB_36_GBIN4), U4.16 (B6)
- new net a4: U10.33 (IOB_35_GBIN5), U4.17 (B5)
- new net a5: U10.36 (IOB_34), U4.18 (B4)
- new net a6: U10.30 (IOB_30), U4.19 (B3)
- new net a7: U10.29 (IOB_29), U4.20 (B2)
- new net ab10: U10.15 (IOL_7A_GBIN6), U5.16 (B6)
- new net ab11: U10.12 (IOL_6A), U5.17 (B5)
- new net ab12: U10.13 (IOL_6B_GBIN7), U5.18 (B4)
- new net ab13: U10.10 (IOL_5B), U5.19 (B3)
- new net ab14: U10.9 (IOL_5A), U5.20 (B2)
- new net ab15: U10.8 (IOL_3B), U5.21 (B1)
- new net ab8: U10.19 (IOL_8B), U5.14 (B8)
- new net ab9: U10.16 (IOL_7B), U5.15 (B7)
- new net as: U10.2 (IOL_1B), U8.17 (B5)
- new net b: U10.4 (IOL_2B), U8.15 (B7)
- new net c: U10.7 (IOL_3A), U8.14 (B8)
- new net d0: U10.28 (IOB_28), U7.14 (B8)
- new net d1: U10.27 (IOB_27), U7.15 (B7)
- new net d2: U10.26 (IOB_26), U7.16 (B6)
- new net d3: U10.25 (IOL_12B), U7.17 (B5)
- new net d4: U10.24 (IOL_12A), U7.18 (B4)
- new net d5: U10.21 (IOL_10B), U7.19 (B3)
- new net d6: U10.20 (IOL_10A), U7.20 (B2)
- new net d7: U10.18 (IOL_8A), U7.21 (B1)
- new net dtack: U1.5, U10.90 (IOT_85_GBIN0)
- new net exreset: U10.99 (IOT_93), U8.20 (B2)
- new net iack2: U10.96 (IOT_90), U9.21 (B1)
- new net iack4: U10.95 (IOT_89), U9.20 (B2)
- new net iddir: U10.94 (IOT_88), U9.19 (B3)
- new net irq2: U1.1, U10.93 (IOT_87)
- new net irq4: U1.3, U10.91 (IOT_86)
- new net lds: U10.1 (IOL_1A), U8.18 (B4)
- new net reset: J2.10 (~RESET~), R3.1, U10.44 (CRESET_B)
- new net rw: U10.100 (IOT_95), U8.19 (B3)
- new net sck: J2.4 (SWDCLK/TCK), U10.49 (IOB_47_SS), U2.1 (~CS)
- new net si: J2.8 (NC/TDI), U10.45 (IOB_44_SDO), U2.5 (SI/IO0)
- new net so: J2.6 (SWO/TDO), U10.46 (IOB_45_SDI), U2.2 (SO/IO1)
- new net ss: J2.2 (SWDIO/TMS), U10.48 (IOB_46_SCK), U2.6 (SCK)
Other:
- moved on the sheet: J3, J7, R6, R9

Commit message: route board
Parts:
- removed R1, R2: 1, Resistor_SMD:R_0805_2012Metric, symbol Device:R
- H1, H2: footprint (none) -> MountingHole:MountingHole_3.2mm_M3_Pad
- J1: symbol x68k:x68000_expansion -> midiori-rescue:x68000_expansion-x68k
- J2: symbol Connector:Conn_ARM_JTAG_SWD_10 -> midiori-rescue:Conn_ARM_JTAG_SWD_10-Connector
- U10: symbol ICE40HX1K-VQ100:ICE40HX1K-VQ100 -> midiori-rescue:ICE40HX1K-VQ100-ICE40HX1K-VQ100
- U11: value TPS76933 -> TPS70933
- U3: value TPS76912 -> TPS70912
- U4, U5, U6, U7, U8, U9: symbol SN74LVC8T245DWR:SN74LVC8T245DWR -> midiori-rescue:SN74LVC8T245DWR-SN74LVC8T245DWR
- X1: symbol x68k:SG5032CAN -> midiori-rescue:SG5032CAN-x68k
Connections:
- net GND: now also C1.2, C2.2, U11.2 (GND), U11.3 (~EN~), U3.2 (GND), U3.3 (~EN~)
- net a16: now also U10.81 (IOT_77); no longer U10.71 (IOR_69)
- net a17: now also U10.80 (IOT_75); no longer U10.72 (IOR_70)
- net a18: now also U10.79 (IOT_74); no longer U10.73 (IOR_71)
- net a19: now also U10.78 (IOT_73); no longer U10.74 (IOR_72)
- net a20: now also U10.74 (IOR_72); no longer U10.78 (IOT_73)
- net a21: now also U10.73 (IOR_71); no longer U10.79 (IOT_74)
- net a22: now also U10.72 (IOR_70); no longer U10.80 (IOT_75)
- net a23: now also U10.71 (IOR_69); no longer U10.81 (IOT_77)
- net a3: now also U10.36 (IOB_34); no longer U10.34 (IOB_36_GBIN4)
- net a4: now also U10.34 (IOB_36_GBIN4); no longer U10.33 (IOB_35_GBIN5)
- net a5: now also U10.33 (IOB_35_GBIN5); no longer U10.36 (IOB_34)
- net ab11: now also U10.13 (IOL_6B_GBIN7); no longer U10.12 (IOL_6A)
- net ab12: now also U10.12 (IOL_6A); no longer U10.13 (IOL_6B_GBIN7)
- net ab8: now also U10.18 (IOL_8A); no longer U10.19 (IOL_8B)
- net d7: now also U10.19 (IOL_8B); no longer U10.18 (IOL_8A)
- net dtack: now also U10.93 (IOT_87); no longer U10.90 (IOT_85_GBIN0)
- net iack2: now also U10.94 (IOT_88); no longer U10.96 (IOT_90)
- net iddir: now also U10.96 (IOT_90); no longer U10.94 (IOT_88)
- net irq2: now also U10.90 (IOT_85_GBIN0); no longer U10.93 (IOT_87)
Changed lines of the file:
@@
-EESchema Schematic File Version 4
+EESchema Schematic File Version 5
 LIBS:midiori-cache
 EELAYER 29 0
@@
 $EndDescr
 $Comp
-L x68k:x68000_expansion J1
+L midiori-rescue:x68000_expansion-x68k J1
 U 1 1 5BFF029F
 P 2150 -1050
@@
 Connection ~ 6550 9750
 $Comp
-L x68k:SG5032CAN X1
+L midiori-rescue:SG5032CAN-x68k X1
 U 1 1 5C01CB41
 P 6550 9450
@@
 	14350 2500 14750 2500
 $Comp
-L SN74LVC8T245DWR:SN74LVC8T245DWR U4
+L midiori-rescue:SN74LVC8T245DWR-SN74LVC8T245DWR U4
 U 1 1 5CB81A7A
 P 4550 1600
@@
 AB7
 $Comp
-L SN74LVC8T245DWR:SN74LVC8T245DWR U5
+L midiori-rescue:SN74LVC8T245DWR-SN74LVC8T245DWR U5
 U 1 1 5CB84A17
 P 4550 3200
@@
 AB15
 $Comp
-L SN74LVC8T245DWR:SN74LVC8T245DWR U6
+L midiori-rescue:SN74LVC8T245DWR-SN74LVC8T245DWR U6
 U 1 1 5CB8623F
 P 4550 4800
@@
 IRQ4
 $Comp
-L SN74LVC8T245DWR:SN74LVC8T245DWR U8
+L midiori-rescue:SN74LVC8T245DWR-SN74LVC8T245DWR U8
 U 1 1 5CB8F4D5
 P 4550 8000
@@
 C
 $Comp
-L SN74LVC8T245DWR:SN74LVC8T245DWR U9
+L midiori-rescue:SN74LVC8T245DWR-SN74LVC8T245DWR U9
 U 1 1 5CB9618A
 P 4550 9600
@@
 IDDIR
 $Comp
-L ICE40HX1K-VQ100:ICE40HX1K-VQ100 U10
+L midiori-rescue:ICE40HX1K-VQ100-ICE40HX1K-VQ100 U10
 U 1 1 5CBA3357
 P 8650 4600
@@
 F 0 "H1" H 14050 7146 50  0000 L CNN
 F 1 "MountingHole" H 14050 7055 50  0000 L CNN
-F 2 "" H 13950 7100 50  0001 C CNN
+F 2 "MountingHole:MountingHole_3.2mm_M3_Pad" H 13950 7100 50  0001 C CNN
 F 3 "~" H 13950 7100 50  0001 C CNN
 	1    13950 7100
@@
 F 0 "H2" H 15050 7146 50  0000 L CNN
 F 1 "MountingHole" H 15050 7055 50  0000 L CNN
-F 2 "" H 14950 7100 50  0001 C CNN
+F 2 "MountingHole:MountingHole_3.2mm_M3_Pad" H 14950 7100 50  0001 C CNN
 F 3 "~" H 14950 7100 50  0001 C CNN
 	1    14950 7100
@@
 Text Label 4650 5100 0    50   ~ 0
 a16
-Text Label 9650 4700 0    50   ~ 0
-a23
-Text Label 9650 4800 0    50   ~ 0
-a22
-Text Label 9650 4900 0    50   ~ 0
-a21
-Text Label 9650 5000 0    50   ~ 0
-a20
-Text Label 9650 5200 0    50   ~ 0
-a19
-Text Label 9650 5300 0    50   ~ 0
-a18
-Text Label 9650 5400 0    50   ~ 0
-a17
-Text Label 9650 5500 0    50   ~ 0
-a16
 Text Label 7550 5500 0    50   ~ 0
 a7
 Text Label 7550 5600 0    50   ~ 0
 a6
-Text Label 7550 5700 0    50   ~ 0
-a5
-Text Label 7550 5800 0    50   ~ 0
-a4
-Text Label 7550 5900 0    50   ~ 0
-a3
 Text Label 7550 6000 0    50   ~ 0
 a2
@@
 Text Label 4650 6700 0    50   ~ 0
 d0
-Text Label 7550 4500 0    50   ~ 0
-d7
 Text Label 7550 4600 0    50   ~ 0
 d6
@@
 Text Label 4650 2800 0    50   ~ 0
 ab15
-Text Label 7450 4400 0    50   ~ 0
-ab8
 Text Label 7450 4300 0    50   ~ 0
 ab9
 Text Label 7450 4200 0    50   ~ 0
 ab10
-Text Label 7450 4100 0    50   ~ 0
-ab11
-Text Label 7450 4000 0    50   ~ 0
-ab12
 Text Label 7450 3900 0    50   ~ 0
 ab13
@@
 Text Label 4650 9400 0    50   ~ 0
 iddir
-Text Label 9650 3500 0    50   ~ 0
-iack2
-Text Label 9650 3600 0    50   ~ 0
-iack4
-Text Label 9650 3700 0    50   ~ 0
-iddir
 Wire Wire Line
 	9650 5800 12450 5800
@@
 irq4
 Text Label 2150 10050 0    50   ~ 0
-dtack
-Text Label 9650 3800 0    50   ~ 0
-irq2
-Text Label 9650 3900 0    50   ~ 0
-irq4
-Text Label 9650 4000 0    50   ~ 0
 dtack
 Wire Wire Line
@@
 P 14900 4500
 F 0 "U3" H 14900 4842 50  0000 C CNN
-F 1 "TPS76912" H 14900 4751 50  0000 C CNN
+F 1 "TPS70912" H 14900 4751 50  0000 C CNN
 F 2 "Package_TO_SOT_SMD:SOT-23-5" H 14900 4825 50  0001 C CIN
 F 3 "http://www.ti.com/lit/ds/symlink/tps769.pdf" H 14900 4450 50  0001 C CNN
@@
 P 13650 4500
 F 0 "U11" H 13650 4842 50  0000 C CNN
-F 1 "TPS76933" H 13650 4751 50  0000 C CNN
+F 1 "TPS70933" H 13650 4751 50  0000 C CNN
 F 2 "Package_TO_SOT_SMD:SOT-23-5" H 13650 4825 50  0001 C CIN
 F 3 "http://www.ti.com/lit/ds/symlink/tps769.pdf" H 13650 4450 50  0001 C CNN
@@
 	1    0    0    -1
 $EndComp
-$Comp
-L Device:R R1
-U 1 1 5CCC388A
-P 14150 4850
-F 0 "R1" H 14220 4896 50  0000 L CNN
-F 1 "1" H 14220 4805 50  0000 L CNN
-F 2 "Resistor_SMD:R_0805_2012Metric" V 14080 4850 50  0001 C CNN
-F 3 "~" H 14150 4850 50  0001 C CNN
-	1    14150 4850
-	1    0    0    -1
-$EndComp
-$Comp
-L Device:R R2
-U 1 1 5CCC412A
-P 15400 4850
-F 0 "R2" H 15470 4896 50  0000 L CNN
-F 1 "1" H 15470 4805 50  0000 L CNN
-F 2 "Resistor_SMD:R_0805_2012Metric" V 15330 4850 50  0001 C CNN
-F 3 "~" H 15400 4850 50  0001 C CNN
-	1    15400 4850
-	1    0    0    -1
-$EndComp
 Wire Wire Line
 	14150 5050 13650 5050
 Wire Wire Line
 	13650 5050 13650 4800
-Wire Wire Line
-	14150 5000 14150 5050
-Wire Wire Line
-	15400 5000 15400 5050
 Connection ~ 14150 5050
 Wire Wire Line
@@
 Connection ~ 14500 5050
 Wire Wire Line
-	14500 5050 14150 5050
+	14500 5050 14300 5050
 Wire Wire Line
 	15300 4400 15400 4400
@@
 	7650 3000 6900 3000
 $Comp
-L Connector:Conn_ARM_JTAG_SWD_10 J2
+L midiori-rescue:Conn_ARM_JTAG_SWD_10-Connector J2
 U 1 1 5CD4062E
 P 8500 8400
@@
 Connection ~ 3650 3700
 $Comp
-L SN74LVC8T245DWR:SN74LVC8T245DWR U7
+L midiori-rescue:SN74LVC8T245DWR-SN74LVC8T245DWR U7
 U 1 1 5CB89CCF
 P 4550 6400
@@
 $EndComp
 $Comp
-L power:+3V3 #PWR?
+L power:+3V3 #PWR0121
 U 1 1 5CE95695
 P 6550 9150
-F 0 "#PWR?" H 6550 9000 50  0001 C CNN
+F 0 "#PWR0121" H 6550 9000 50  0001 C CNN
 F 1 "+3V3" H 6565 9323 50  0000 C CNN
 F 2 "" H 6550 9150 50  0001 C CNN
@@
 $EndComp
 Connection ~ 6550 9150
+Text Label 7450 4000 0    50   ~ 0
+ab11
+Text Label 7450 4100 0    50   ~ 0
+ab12
+Text Label 7450 4400 0    50   ~ 0
+d7
+Text Label 7550 4500 0    50   ~ 0
+ab8
+Text Label 7550 5800 0    50   ~ 0
+a5
+Text Label 7550 5900 0    50   ~ 0
+a4
+Text Label 7550 5700 0    50   ~ 0
+a3
+Wire Wire Line
+	14150 4700 14150 5050
+Wire Wire Line
+	15400 4700 15400 5050
+Text Label 9650 3700 0    50   ~ 0
+iack2
+Text Label 9650 3600 0    50   ~ 0
+iack4
+Text Label 9650 3500 0    50   ~ 0
+iddir
+Text Label 9650 3800 0    50   ~ 0
+dtack
+Text Label 9650 3900 0    50   ~ 0
+irq4
+Text Label 9650 4000 0    50   ~ 0
+irq2
+Text Label 9650 4700 0    50   ~ 0
+a16
+Text Label 9650 4800 0    50   ~ 0
+a17
+Text Label 9650 4900 0    50   ~ 0
+a18
+Text Label 9650 5000 0    50   ~ 0
+a19
+Text Label 9650 5200 0    50   ~ 0
+a20
+Text Label 9650 5300 0    50   ~ 0
+a21
+Text Label 9650 5400 0    50   ~ 0
+a22
+Text Label 9650 5500 0    50   ~ 0
+a23
+$Comp
+L power:GND #PWR0151
+U 1 1 5CC3FD20
+P 14300 5050
+F 0 "#PWR0151" H 14300 4800 50  0001 C CNN
+F 1 "GND" H 14305 4877 50  0000 C CNN
+F 2 "" H 14300 5050 50  0001 C CNN
+F 3 "" H 14300 5050 50  0001 C CNN
+	1    14300 5050
+	1    0    0    -1
+$EndComp
+Connection ~ 14300 5050
+Wire Wire Line
+	14300 5050 14150 5050
 $EndSCHEMATC

Commit message: midiori v2.1 pcb
Parts:
- removed U11: TPS70933, Package_TO_SOT_SMD:SOT-23-5, symbol Regulator_Linear:TPS76933
- removed U3: TPS70912, Package_TO_SOT_SMD:SOT-23-5, symbol Regulator_Linear:TPS76912
- added J4: Conn_02x03_Odd_Even, Connector:Tag-Connect_TC2030-IDC-NL_2x03_P1.27mm_Vertical, symbol Connector_Generic:Conn_02x03_Odd_Even
- added unit 5 of U1
- added unit 6 of U1
- added unit 7 of U1
- added U11: TLV73333PDBV, Package_TO_SOT_SMD:SOT-23-5, symbol Regulator_Linear:TLV73333PDBV
- added U3: TLV73312PDBV, Package_TO_SOT_SMD:SOT-23-5, symbol Regulator_Linear:TLV73312PDBV
- J1: symbol midiori-rescue:x68000_expansion-x68k -> midiori-rescue:x68000_expansion-x68k-midiori-rescue
- J2: symbol midiori-rescue:Conn_ARM_JTAG_SWD_10-Connector -> midiori-rescue:Conn_ARM_JTAG_SWD_10-Connector-midiori-rescue
- U10: symbol midiori-rescue:ICE40HX1K-VQ100-ICE40HX1K-VQ100 -> midiori-rescue:ICE40HX1K-VQ100-ICE40HX1K-VQ100-midiori-rescue
- U4, U5, U6, U7, U8, U9: symbol midiori-rescue:SN74LVC8T245DWR-SN74LVC8T245DWR -> midiori-rescue:SN74LVC8T245DWR-SN74LVC8T245DWR-midiori-rescue
- X1: symbol midiori-rescue:SG5032CAN-x68k -> midiori-rescue:SG5032CAN-x68k-midiori-rescue
Connections:
- net +1V2: now also U3.5 (OUT)
- net +3V3: now also J4.1 (Pin_1), U1.14 (VCC), U11.5 (OUT), U3.1 (IN), U3.3 (EN)
- net +5V: now also U4.2 (DIR), U5.2 (DIR), U6.2 (DIR), U8.2 (DIR), U9.2 (DIR), U11.1 (IN), U11.3 (EN)
- net GND: now also U4.21 (B1), U4.22 (OE), U4.3 (A1), U5.22 (OE), U6.22 (OE), U8.22 (OE), U9.10 (A8), U9.14 (B8), U9.15 (B7), U9.16 (B6), U9.17 (B5), U9.18 (B4), U9.22 (OE), U9.6 (A4), U9.7 (A5), U9.8 (A6), U9.9 (A7), J4.5 (Pin_5), U1.11, U1.13, U1.7 (GND), U11.2 (GND), U3.2 (GND)
- net reset: now also J2.8 (NC/TDI); no longer J2.10 (~RESET~)
- net sck: now also J4.4 (Pin_4)
- net si: now also J2.2 (SWDIO/TMS), J4.2 (Pin_2); no longer J2.8 (NC/TDI)
- net so: now also J2.10 (~RESET~), J4.3 (Pin_3); no longer J2.6 (SWO/TDO)
- net ss: now also J2.6 (SWO/TDO), J4.6 (Pin_6); no longer J2.2 (SWDIO/TMS)
- net xltr_oe: now reaches U7.22 (OE)
- net xltr_oe: now also U10.51 (IOR_52)
- no-connect marks 0 -> 2
