File: midiori.sch (KiCad schematic (older format))
At the start: 45 parts, among them J1 x68000_expansion, J2 Conn_ARM_JTAG_SWD_10, J3 DIN-5_180degree, J4 Conn_02x03_Odd_Even, J7 AudioJack3, U1 74LCX07, U10 ICE40HX1K-VQ100, U11 TLV73333PDBV, U2 AT25SF081-SSHD-X, U3 TLV73312PDBV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

Commit message: add more connectors
Parts:
- removed J4: Conn_02x03_Odd_Even, Connector:Tag-Connect_TC2030-IDC-NL_2x03_P1.27mm_Vertical, symbol Connector_Generic:Conn_02x03_Odd_Even
- added J4: Mini-DIN-5, x68k:MD-50SM, symbol Connector:Mini-DIN-5
Connections:
- wire segments 228 -> 235
Other:
- moved on the sheet: R6

Commit message: one connector
Parts:
- removed J3: DIN-5_180degree, x68k:sds-50j, symbol Connector:DIN-5_180degree
- removed J7: AudioJack3, Connector_Audio:Jack_3.5mm_CUI_SJ1-3533NG_Horizontal, symbol Connector:AudioJack3
Connections:
- wire segments 235 -> 238
- no-connect marks 2 -> 4
