File: midiori.kicad_sch (KiCad schematic)
At the start: 94 parts, among them J1 midiori-rescue_x68000_expansi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, J2 Conn_ARM_JTAG_SWD_10, J3 AudioJack3, J4 Mini-DIN-5, J5 AudioJack3, J6 AudioJack3, J7 Conn_01x06, J8 AudioJack3, J9 Mini-DIN-5, U1 74lv07, U10 ICE40HX4K-TQ144, U11 AP2205K-3.3, U12 AK4432, U13 TL072, U14 AP2205K-3.3, U15 TL072, U16 74lv07, U17 H11L1, U18 SN74LVC245APW, U19 74lv07, U2 AT25SF081-SSHD-X, U3 AP2127K-1.2, U4 SN74LVC245APW, U5 SN74LVC245APW, U6 SN74LVC245APW, U7 SN74LVC245APW, U8 SN74LVC245APW, U9 SN74LVC245APW, X1 16MHz, X2 24.576MHz

Commit message: add ram
Parts:
- added C42: 0.1uF, Capacitor_SMD:C_0805_2012Metric, symbol Device:C
- added U20: IS66WVE4M16TBLL-70BLI, Package_BGA:TFBGA-48_6x10mm_Layout6x8_P0.75mm, symbol x68k:IS66WVE4M16TBLL-70BLI
Connections:
- net +3V3: now also C42.1, U20.D6 (VDD), U20.E1 (VDDQ)
- net GND: now also C42.2, U20.D1 (VSSQ), U20.E6 (VSS)
- net a16: now also U20.F4 (A15)
- net a17: now also U20.E4 (A16)
- net a18: now also U20.D3 (A17)
- net a19: now also U20.H1 (A18)
- net a20: now also U20.G2 (A19)
- net a21: now also U20.H6 (A20)
- net a22: now also U20.E3 (A21)
- net ab10: now also U20.H3 (A9)
- net ab11: now also U20.H4 (A10)
- net ab12: now also U20.H5 (A11)
- net ab13: now also U20.G3 (A12)
- net ab14: now also U20.G4 (A13)
- net ab15: now also U20.F3 (A14)
- net ab8: now also U20.D4 (A7)
- net ab9: now also U20.H2 (A8)
- net d0: now also U20.B6 (DQ0)
- net d1: now also U20.C5 (DQ1)
- net d2: now also U20.C6 (DQ2)
- net d3: now also U20.D5 (DQ3)
- net d4: now also U20.E5 (DQ4)
- net d5: now also U20.F5 (DQ5)
- net d6: now also U20.F6 (DQ6)
- net d7: now also U20.G6 (DQ7)
- net db10: now also U20.C2 (DQ10)
- net db11: now also U20.D2 (DQ11)
- net db12: now also U20.E2 (DQ12)
- net db13: now also U20.F2 (DQ13)
- net db14: now also U20.F1 (DQ14)
- net db15: now also U20.G1 (DQ15)
- net db8: now also U20.B1 (DQ8)
- net db9: now also U20.C1 (DQ9)
- net lds: now also U20.A1 (~{LB})
- net rw: now also U20.G5 (~{WE})
- net uds: now also U20.B2 (~{UB})
- net ~{ram_oe}: now reaches U10.33 (IOL_25A)
- net ~{ram_oe}: now also U20.A2 (~{OE})
- net ~{ram_ce}: now reaches U10.34 (IOL_25B)
- net ~{ram_ce}: now also U20.B5 (~{CE})
- new net +3.3V: U20.A6 (~{ZZ})
- new net ab1: U20.A3 (A0)
- new net ab2: U20.A4 (A1)
- new net ab3: U20.A5 (A2)
- new net ab4: U20.B3 (A3)
- new net ab5: U20.B4 (A4)
- new net ab6: U20.C3 (A5)
- new net ab7: U20.C4 (A6)

Commit message: Add muting circuit, remove a lv07, rearrange
Parts:
- removed TP1, TP2: TestPoint, TestPoint:TestPoint_THTPad_1.0x1.0mm_Drill0.5mm, symbol Connector:TestPoint
- removed unit 2 of U16
- removed unit 1 of U16
- removed unit 3 of U16
- removed unit 5 of U16
- removed unit 6 of U16
- removed unit 4 of U16
- added C43: 0.1uF, Capacitor_SMD:C_0805_2012Metric, symbol Device:C
- added Q1, Q2: MMBFJ111, Package_TO_SOT_SMD:SOT-23, symbol Transistor_FET:MMBFJ111
- added R18: 10k, symbol Device:R
- added R19: 1k, Resistor_SMD:R_0805_2012Metric, symbol Device:R
- added R20: 10k, Resistor_SMD:R_0805_2012Metric, symbol Device:R
- added SW1: SW_DIP_x03, Package_BGA:TFBGA-48_6x10mm_Layout6x8_P0.75mm, symbol Switch:SW_DIP_x03
- added U21: SN74LVC245APW, Package_SO:SOIC-20W_7.5x12.8mm_P1.27mm, symbol Logic_LevelTranslator:SN74LVC245APW
Connections:
- net CBSEL1 is gone; now on net GND: U10.64 (IOB_104_CBSEL1)
- net +3.3V: now also SW1.4
- net +3V3: now also U21.20 (VCC)
- net -12V: now also R19.1
- net 20MHz: now also U8.8 (A7); no longer U18.3 (A2)
- net 20mhz: now also U10.142 (IOT_220), U8.12 (B7); no longer U18.17 (B2)
- net AS: now also U21.6 (A5); no longer U8.8 (A7)
- net DTACK: now also U19.10
- net EXREQ: now also U19.12
- net GND: now also U18.17 (B2), U18.3 (A2), C43.2, Q1.2 (S), Q2.2 (S), R18.2, R20.1, SW1.5, SW1.6, U21.10 (GND), U21.19 (~{OE}); no longer U19.11, U19.13
- net LDS: now also U21.7 (A6); no longer U8.7 (A6)
- net RW: now also U21.9 (A8); no longer U8.5 (A4)
- net UDS: now also U21.8 (A7); no longer U8.6 (A5)
- net addr_dir: now also U21.1 (DIR)
- net as: now also U21.14 (B5); no longer U8.12 (B7)
- net dtack_drv: now also U19.11
- net exreq_drv: now also U19.13
- net lds: now also U21.13 (B6); no longer U8.13 (B6)
- net rw: now also U21.11 (B8); no longer U8.15 (B4)
- net uds: now also U21.12 (B7); no longer U8.14 (B5)
- net dip1: now reaches U10.31 (IOL_24A)
- net dip1: now also SW1.1
- net dip2: now reaches U10.32 (IOL_24B)
- net dip2: now also SW1.2
- net at C32.2, R13.2: now also Q2.1 (D)
- net at C31.2, R12.2: now also Q1.1 (D)
- net CBSEL0 renamed cbsel0
- net cbsel0: now also R18.1, SW1.3
- net as_drv: no longer names the net of U10.121 (IOT_181)
- net lds_drv: no longer names the net of U10.120 (IOT_179)
- net rw_drv: no longer names the net of U10.118 (IOT_177)
- net uds_drv: no longer names the net of U10.119 (IOT_178)
- new net: C43.1, Q1.3 (G), Q2.3 (G), R19.2, R20.2
- no-connect marks 40 -> 44
Other:
- moved on the sheet: C13, C24, C29, C30, C31, C32, C33, C34, C35, C37, C41, C42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

Commit message: lots of stuff
Parts:
- removed JP1: ACKS, Jumper:SolderJumper-3_P1.3mm_Bridged12_Pad1.0x1.5mm, symbol Jumper:Jumper_3_Bridged12
- removed JP2: DIF, Jumper:SolderJumper-3_P1.3mm_Bridged12_Pad1.0x1.5mm, symbol Jumper:Jumper_3_Bridged12
- removed U16: 74lv07, Package_SO:SOIC-14_3.9x8.7mm_P1.27mm, symbol 74xx:74LCX07
- SW1: footprint Package_BGA:TFBGA-48_6x10mm_Layout6x8_P0.75mm -> Button_Switch_SMD:SW_DIP_SPSTx03_Slide_9.78x9.8mm_W8.61mm_P2.54mm
Connections:
- net +3.3V is gone; now on net +3V3: SW1.4, U20.A6 (~{ZZ})
- net ab1 is gone; now on net a1: U20.A3 (A0)
- net ab2 is gone; now on net a2: U20.A4 (A1)
- net ab3 is gone; now on net a3: U20.A5 (A2)
- net ab4 is gone; now on net a4: U20.B3 (A3)
- net ab5 is gone; now on net a5: U20.B4 (A4)
- net ab6 is gone; now on net a6: U20.C3 (A5)
- net ab7 is gone; now on net a7: U20.C4 (A6)
- net +3V3: now also U12.7 (ACKS/CCLK/SCL), U12.8 (DIF/CDTI/SDA)
- net 10m: now also U10.137 (IOT_215); no longer U10.141 (IOT_219)
- net 16mhz: now also U10.96 (IOR_146); no longer U10.88 (IOR_137)
- net 20mhz: now also U10.136 (IOT_214); no longer U10.142 (IOT_220)
- net 24.576mhz: now also U10.95 (IOR_144); no longer U10.87 (IOR_136)
- net AS: now also U21.9 (A8); no longer U21.6 (A5)
- net BG: now also U18.4 (A3); no longer U18.5 (A4)
- net BGACK: now also U18.3 (A2); no longer U18.4 (A3)
- net GND: no longer U18.17 (B2), U18.3 (A2)
- net IACK2: now also U18.6 (A5); no longer U18.7 (A6)
- net IACK4: now also U18.5 (A4); no longer U18.6 (A5)
- net LDS: now also U21.8 (A7); no longer U21.7 (A6)
- net RW: now also U21.6 (A5); no longer U21.9 (A8)
- net UDS: now also U21.7 (A6); no longer U21.8 (A7)
- net a21: no longer U20.H6 (A20)
- net a22: no longer U20.E3 (A21)
- net ab10: now also U10.32 (IOL_24B); no longer U10.26 (IOL_18B)
- net ab11: now also U10.31 (IOL_24A); no longer U10.25 (IOL_18A)
- net ab8: now also U10.34 (IOL_25B); no longer U10.29 (IOL_23B)
- net ab9: now also U10.33 (IOL_25A); no longer U10.28 (IOL_23A)
- net addr_dir: now also U10.26 (IOL_18B); no longer U10.62 (IOB_102)
- net as: now also U10.142 (IOT_220), U21.11 (B8); no longer U10.139 (IOT_217), U21.14 (B5)
- net bg: now also U10.121 (IOT_181), U18.16 (B3); no longer U10.122 (IOT_190), U18.15 (B4)
- net bgack: now also U10.120 (IOT_179), U18.17 (B2); no longer U10.101 (IOR_160), U18.16 (B3)
- net bick: now also U10.81 (IOR_117); no longer U10.76 (IOR_112)
- net data_dir: now also U10.28 (IOL_23A); no longer U10.61 (IOB_96)
- net dip1: now also U10.73 (IOR_109); no longer U10.31 (IOL_24A)
- net dip2: now also U10.74 (IOR_110); no longer U10.32 (IOL_24B)
- net dtack_drv: now also U10.118 (IOT_177); no longer U10.117 (IOT_174)
- net exreq_drv: now also U10.117 (IOT_174); no longer U10.116 (IOT_173)
- net iack2: now also U10.124 (IOT_191), U18.14 (B5); no longer U10.125 (IOT_192), U18.13 (B6)
- net iack4: now also U10.122 (IOT_190), U18.15 (B4); no longer U10.124 (IOT_191), U18.14 (B5)
- net lds: now also U10.141 (IOT_219), U21.12 (B7); no longer U10.138 (IOT_216), U21.13 (B6)
- net lrck: now also U10.79 (IOR_115); no longer U10.74 (IOR_110)
- net midi_in: now also U10.104 (IOR_164); no longer U10.98 (IOR_148)
- net midi_out: now also U10.105 (IOR_165); no longer U10.99 (IOR_152)
- net rw: now also U10.138 (IOT_216), U21.14 (B5); no longer U10.136 (IOT_214), U21.11 (B8)
- net sdti: now also U10.80 (IOR_116); no longer U10.75 (IOR_111)
- net smute: now also U10.78 (IOR_114); no longer U10.73 (IOR_109)
- net uds: now also U10.139 (IOT_217), U21.13 (B6); no longer U10.137 (IOT_215), U21.12 (B7)
- net xltr_oe: now also U10.25 (IOL_18A); no longer U10.78 (IOR_114)
- net ~{ram_ce}: now also U10.76 (IOR_112); no longer U10.34 (IOL_25B)
- net ~{ram_oe}: now also U10.75 (IOR_111); no longer U10.33 (IOL_25A)
- net EXBERR: now reaches J1.A39
- net EXBERR: now also U18.7 (A6)
- new net exberr: U10.125 (IOT_192), U18.13 (B6)
- new net ram_a21: U10.61 (IOB_96), U20.H6 (A20)
- new net ram_a22: U10.62 (IOB_102), U20.E3 (A21)
- no-connect marks 44 -> 60
Other:
- moved on the sheet: H1, H2
